Commit message: feat: each tf tree build success.

File: hive_gazebo/urdf/_d435i.urdf.xacro (robot description, xacro)
@@ -20,7 +20,7 @@
 -->
 <robot name="sensor_d435i" xmlns:xacro="http://ros.org/wiki/xacro">
-  <xacro:include filename="$(find realsense2_description)/urdf/_d435.urdf.xacro"/>
-  <xacro:include filename="$(find realsense2_description)/urdf/_d435i_imu_modules.urdf.xacro"/>
-  <xacro:macro name="sensor_d435i" params="parent *origin name:=camera use_nominal_extrinsics:=false">
+  <xacro:include filename="$(find hive_gazebo)/urdf/_d435.urdf.xacro"/>
+  <xacro:include filename="$(find hive_gazebo)/urdf/_d435i_imu_modules.urdf.xacro"/>
+  <xacro:macro name="sensor_d435i" params="parent *origin name:=camera1 use_nominal_extrinsics:=false">
     <xacro:sensor_d435 parent="${parent}" name="${name}" use_nominal_extrinsics="${use_nominal_extrinsics}">
       <xacro:insert_block name="origin" />

File: hive_gazebo/urdf/test_d435i_camera.urdf.xacro (robot description, xacro)
@@ -2,7 +2,7 @@
 <robot name="realsense2_camera" xmlns:xacro="http://www.ros.org/wiki/xacro">
   <xacro:arg name="use_nominal_extrinsics" default="false" />
-  <xacro:include filename="$(find realsense2_description)/urdf/_d435i.urdf.xacro"/>
-  <link name="base_link" />
-  <xacro:sensor_d435i parent="base_link" use_nominal_extrinsics="$(arg use_nominal_extrinsics)">
+  <xacro:include filename="$(find hive_gazebo)/urdf/_d435i.urdf.xacro"/>
+  <link name="ceiling_link" />
+  <xacro:sensor_d435i parent="ceiling_link" use_nominal_extrinsics="$(arg use_nominal_extrinsics)">
     <origin xyz="0 0 0" rpy="0 0 0"/>
   </xacro:sensor_d435i>
