Commit message: feat(hive_gazebo) add diff controller

File: hive_gazebo/urdf/geunwoo.xacro (robot description, xacro)
@@ -7,5 +7,6 @@
   <inertial>
     <origin xyz="-0.10589890450472451 0.004101721807053668 0.2428453449181509" rpy="0 0 0"/>
-    <mass value="97.68742911120015"/>
+    <!-- <mass value="97.68742911120015"/> -->
+    <mass value="40.0"/>
     <inertia ixx="5.633563" iyy="4.887417" izz="5.433869" ixy="0.000389" iyz="-0.000239" ixz="0.200866"/>
   </inertial>
@@ -114,5 +115,5 @@
   <parent link="base_link"/>
   <child link="right_wheel"/>
-  <axis xyz="-0.0 -1.0 -0.0"/>
+  <axis xyz="0.0 1.0 0.0"/>
 </joint>
 <joint name="right_caster_joint" type="continuous">

Commit message: style:

File: hive_gazebo/urdf/geunwoo.xacro (robot description, xacro)
@@ -3,5 +3,5 @@
 <xacro:include filename="$(find hive_gazebo)/urdf/materials.xacro" />
 <xacro:include filename="$(find hive_gazebo)/urdf/geunwoo.trans" />
-<xacro:include filename="$(find hive_gazebo)/urdf/geunwoo.gazebo" />
+<xacro:include filename="$(find hive_gazebo)/urdf/geunwoo_gazebo.xacro" />
 <link name="base_link">
   <inertial>

File: hive_gazebo/urdf/test_d435i_camera.urdf.xacro (robot description, xacro)
@@ -3,7 +3,10 @@
   <xacro:arg name="use_nominal_extrinsics" default="false" />
   <xacro:include filename="$(find hive_gazebo)/urdf/_d435i.urdf.xacro"/>
-  <link name="ceiling_link" />
+   <xacro:property name="M_PI" value="3.1415926535897931" />
+  <link name="ceiling_link">
+    <origin xyz="0 0 0" rpy="0 0 0"/>
+  </link>
   <xacro:sensor_d435i parent="ceiling_link" use_nominal_extrinsics="$(arg use_nominal_extrinsics)">
-    <origin xyz="0 0 0" rpy="0 0 0"/>
+    <origin xyz="1 1 0" rpy="0 0 0"/>
   </xacro:sensor_d435i>
 </robot>
