Commit message: style: devide package in two directory.

File: hive_description/urdf/_d435.urdf.xacro (robot description, xacro)
@@ -21,6 +21,6 @@
 <robot name="sensor_d435" xmlns:xacro="http://ros.org/wiki/xacro">
   <!-- Includes -->
-  <xacro:include filename="$(find hive_gazebo)/urdf/_materials.urdf.xacro" />
-  <xacro:include filename="$(find hive_gazebo)/urdf/_usb_plug.urdf.xacro" />
+  <xacro:include filename="$(find hive_description)/urdf/_materials.urdf.xacro" />
+  <xacro:include filename="$(find hive_description)/urdf/_usb_plug.urdf.xacro" />
   <xacro:macro name="sensor_d435" params="parent *origin name:=camera1 use_nominal_extrinsics:=false add_plug:=false use_mesh:=true">
     <xacro:property name="M_PI" value="3.1415926535897931" />

File: hive_description/urdf/_d435i.urdf.xacro (robot description, xacro)
@@ -20,6 +20,6 @@
 -->
 <robot name="sensor_d435i" xmlns:xacro="http://ros.org/wiki/xacro">
-  <xacro:include filename="$(find hive_gazebo)/urdf/_d435.urdf.xacro"/>
-  <xacro:include filename="$(find hive_gazebo)/urdf/_d435i_imu_modules.urdf.xacro"/>
+  <xacro:include filename="$(find hive_description)/urdf/_d435.urdf.xacro"/>
+  <xacro:include filename="$(find hive_description)/urdf/_d435i_imu_modules.urdf.xacro"/>
   <xacro:macro name="sensor_d435i" params="parent *origin name:=camera1 use_nominal_extrinsics:=false">
     <xacro:sensor_d435 parent="${parent}" name="${name}" use_nominal_extrinsics="${use_nominal_extrinsics}">

File: hive_description/urdf/geunwoo.xacro (robot description, xacro)
@@ -1,7 +1,7 @@
 <?xml version="1.0" ?>
 <robot name="geunwoo" xmlns:xacro="http://www.ros.org/wiki/xacro">
-<xacro:include filename="$(find hive_gazebo)/urdf/materials.xacro" />
-<xacro:include filename="$(find hive_gazebo)/urdf/geunwoo.trans" />
-<xacro:include filename="$(find hive_gazebo)/urdf/geunwoo_gazebo.xacro" />
+<xacro:include filename="$(find hive_description)/urdf/materials.xacro" />
+<xacro:include filename="$(find hive_description)/urdf/geunwoo.trans" />
+<xacro:include filename="$(find hive_description)/urdf/geunwoo_gazebo.xacro" />
 <link name="base_link">
   <inertial>
@@ -14,5 +14,5 @@
     <origin xyz="0 0 0" rpy="0 0 0"/>
     <geometry>
-      <mesh filename="file://$(find hive_gazebo)/meshes/base_link.stl" scale="0.001 0.001 0.001"/>
+      <mesh filename="file://$(find hive_description)/meshes/base_link.stl" scale="0.001 0.001 0.001"/>
     </geometry>
     <material name="silver"/>
@@ -21,5 +21,5 @@
     <origin xyz="0 0 0" rpy="0 0 0"/>
     <geometry>
-      <mesh filename="file://$(find hive_gazebo)/meshes/base_link.stl" scale="0.001 0.001 0.001"/>
+      <mesh filename="file://$(find hive_description)/meshes/base_link.stl" scale="0.001 0.001 0.001"/>
     </geometry>
   </collision>
@@ -34,5 +34,5 @@
     <origin xyz="1e-06 -0.277578 0.0" rpy="0 0 0"/>
     <geometry>
-      <mesh filename="file://$(find hive_gazebo)/meshes/left_wheel_1.stl" scale="0.001 0.001 0.001"/>
+      <mesh filename="file://$(find hive_description)/meshes/left_wheel_1.stl" scale="0.001 0.001 0.001"/>
     </geometry>
     <material name="silver"/>
@@ -41,5 +41,5 @@
     <origin xyz="1e-06 -0.277578 0.0" rpy="0 0 0"/>
     <geometry>
-      <mesh filename="file://$(find hive_gazebo)/meshes/left_wheel_1.stl" scale="0.001 0.001 0.001"/>
+      <mesh filename="file://$(find hive_description)/meshes/left_wheel_1.stl" scale="0.001 0.001 0.001"/>
     </geometry>
   </collision>
@@ -54,5 +54,5 @@
     <origin xyz="1e-06 0.269222 0.0" rpy="0 0 0"/>
     <geometry>
-      <mesh filename="file://$(find hive_gazebo)/meshes/right_wheel_1.stl" scale="0.001 0.001 0.001"/>
+      <mesh filename="file://$(find hive_description)/meshes/right_wheel_1.stl" scale="0.001 0.001 0.001"/>
     </geometry>
     <material name="silver"/>
@@ -61,5 +61,5 @@
     <origin xyz="1e-06 0.269222 0.0" rpy="0 0 0"/>
     <geometry>
-      <mesh filename="file://$(find hive_gazebo)/meshes/right_wheel_1.stl" scale="0.001 0.001 0.001"/>
+      <mesh filename="file://$(find hive_description)/meshes/right_wheel_1.stl" scale="0.001 0.001 0.001"/>
     </geometry>
   </collision>
@@ -74,5 +74,5 @@
     <origin xyz="0.310001 0.185822 -0.043" rpy="0 0 0"/>
     <geometry>
-      <mesh filename="file://$(find hive_gazebo)/meshes/right_caster_1.stl" scale="0.001 0.001 0.001"/>
+      <mesh filename="file://$(find hive_description)/meshes/right_caster_1.stl" scale="0.001 0.001 0.001"/>
     </geometry>
     <material name="silver"/>
@@ -81,5 +81,5 @@
     <origin xyz="0.310001 0.185822 -0.043" rpy="0 0 0"/>
     <geometry>
-      <mesh filename="file://$(find hive_gazebo)/meshes/right_caster_1.stl" scale="0.001 0.001 0.001"/>
+      <mesh filename="file://$(find hive_description)/meshes/right_caster_1.stl" scale="0.001 0.001 0.001"/>
     </geometry>
   </collision>
@@ -94,5 +94,5 @@
     <origin xyz="0.310001 -0.194178 -0.043" rpy="0 0 0"/>
     <geometry>
-      <mesh filename="file://$(find hive_gazebo)/meshes/left_caster_1.stl" scale="0.001 0.001 0.001"/>
+      <mesh filename="file://$(find hive_description)/meshes/left_caster_1.stl" scale="0.001 0.001 0.001"/>
     </geometry>
     <material name="silver"/>
@@ -101,5 +101,5 @@
     <origin xyz="0.310001 -0.194178 -0.043" rpy="0 0 0"/>
     <geometry>
-      <mesh filename="file://$(find hive_gazebo)/meshes/left_caster_1.stl" scale="0.001 0.001 0.001"/>
+      <mesh filename="file://$(find hive_description)/meshes/left_caster_1.stl" scale="0.001 0.001 0.001"/>
     </geometry>
   </collision>

File: hive_description/urdf/test_d435i_camera.urdf.xacro (robot description, xacro)
@@ -2,5 +2,5 @@
 <robot name="realsense2_camera" xmlns:xacro="http://www.ros.org/wiki/xacro">
   <xacro:arg name="use_nominal_extrinsics" default="false" />
-  <xacro:include filename="$(find hive_gazebo)/urdf/_d435i.urdf.xacro"/>
+  <xacro:include filename="$(find hive_description)/urdf/_d435i.urdf.xacro"/>
    <xacro:property name="M_PI" value="3.1415926535897931" />
   <link name="ceiling_link">
