Commit message: feat: add diff controller

File: hive_description/urdf/geunwoo.xacro (robot description, xacro)
@@ -4,5 +4,6 @@
 <xacro:include filename="$(find hive_description)/urdf/geunwoo.trans" />
 <xacro:include filename="$(find hive_description)/urdf/geunwoo_gazebo.xacro" />
-<link name="base_link">
+<xacro:arg name="robot_name" default="robot_1"/>
+<link name="$(arg robot_name)_base_link">
   <inertial>
     <origin xyz="-0.10589890450472451 0.004101721807053668 0.2428453449181509" rpy="0 0 0"/>
@@ -25,5 +26,5 @@
   </collision>
 </link>
-<link name="left_wheel">
+<link name="$(arg robot_name)_left_wheel">
   <inertial>
     <origin xyz="2.6594023369474935e-07 -0.006200652298741449 -4.894162568547244e-09" rpy="0 0 0"/>
@@ -45,5 +46,5 @@
   </collision>
 </link>
-<link name="right_wheel">
+<link name="$(arg robot_name)_right_wheel">
   <inertial>
     <origin xyz="2.5883027950490597e-07 0.006201095560612602 -2.8975644106310483e-10" rpy="0 0 0"/>
@@ -65,5 +66,5 @@
   </collision>
 </link>
-<link name="right_caster">
+<link name="$(arg robot_name)_right_caster">
   <inertial>
     <origin xyz="-0.017519612985357313 2.0677910783639675e-07 -0.05240105157186727" rpy="0 0 0"/>
@@ -85,5 +86,5 @@
   </collision>
 </link>
-<link name="left_caster">
+<link name="$(arg robot_name)_left_caster">
   <inertial>
     <origin xyz="-0.017519612985357313 2.0677910747557426e-07 -0.05240105157186712" rpy="0 0 0"/>
@@ -105,26 +106,26 @@
   </collision>
 </link>
-<joint name="left_wheel_joint" type="continuous">
+<joint name="$(arg robot_name)_left_wheel_joint" type="continuous">
   <origin xyz="-1e-06 0.277578 0.0" rpy="0 0 0"/>
-  <parent link="base_link"/>
-  <child link="left_wheel"/>
+  <parent link="$(arg robot_name)_base_link"/>
+  <child link="$(arg robot_name)_left_wheel"/>
   <axis xyz="0.0 1.0 0.0"/>
 </joint>
-<joint name="right_wheel_joint" type="continuous">
+<joint name="$(arg robot_name)_right_wheel_joint" type="continuous">
   <origin xyz="-1e-06 -0.269222 0.0" rpy="0 0 0"/>
-  <parent link="base_link"/>
-  <child link="right_wheel"/>
+  <parent link="$(arg robot_name)_base_link"/>
+  <child link="$(arg robot_name)_right_wheel"/>
   <axis xyz="0.0 1.0 0.0"/>
 </joint>
-<joint name="right_caster_joint" type="continuous">
+<joint name="$(arg robot_name)_right_caster_joint" type="continuous">
   <origin xyz="-0.310001 -0.185822 0.043" rpy="0 0 0"/>
-  <parent link="base_link"/>
-  <child link="right_caster"/>
+  <parent link="$(arg robot_name)_base_link"/>
+  <child link="$(arg robot_name)_right_caster"/>
   <axis xyz="0.0 0.0 -1.0"/>
 </joint>
-<joint name="left_caster_joint" type="continuous">
+<joint name="$(arg robot_name)_left_caster_joint" type="continuous">
   <origin xyz="-0.310001 0.194178 0.043" rpy="0 0 0"/>
-  <parent link="base_link"/>
-  <child link="left_caster"/>
+  <parent link="$(arg robot_name)_base_link"/>
+  <child link="$(arg robot_name)_left_caster"/>
   <axis xyz="0.0 0.0 -1.0"/>
 </joint>

File: hive_description/urdf/geunwoo_gazebo.xacro (robot description, xacro)
@@ -16,26 +16,4 @@
           <namespace>${robot_name}</namespace>
         </ros>
-      </plugin>
-      <!--diff_drive-->
-      <plugin name='diff_drive' filename='libgazebo_ros_diff_drive.so'>
-        <ros>
-          <!--cmd_vel and odom name remap-->
-          <remapping>cmd_vel:=cmd_vel1</remapping>
-          <remapping>odom:=odom1</remapping>
-        </ros>
-        <!-- Wheel Information -->
-        <left_joint>left_wheel_joint</left_joint>
-        <right_joint>right_wheel_joint</right_joint>
-        <wheel_separation>0.5336</wheel_separation>
-        <wheel_diameter>0.115</wheel_diameter>
-        <!-- Limits -->
-        <max_wheel_torque>200</max_wheel_torque>
-        <max_wheel_acceleration>10.0</max_wheel_acceleration>
-        <!-- Output -->
-        <odometry_frame>odom</odometry_frame>
-        <robot_base_frame>base_link</robot_base_frame>
-        <publish_odom>true</publish_odom>
-        <publish_odom_tf>true</publish_odom_tf>
-        <publish_wheel_tf>true</publish_wheel_tf>
       </plugin>
       <!-- joint -->
