Commit message: fix: one camera description

File: hive_gazebo/urdf/camera1/_d435.urdf.xacro (robot description, xacro)
@@ -19,5 +19,6 @@
 aluminum peripherial evaluation case.
 -->
-<robot name="sensor_d435" xmlns:xacro="http://ros.org/wiki/xacro">
+<robot name="sensor_d435"
+  xmlns:xacro="http://ros.org/wiki/xacro">
   <!-- Includes -->
   <xacro:include filename="$(find hive_gazebo)/urdf/camera1/_materials.urdf.xacro" />
@@ -66,5 +67,5 @@
           <origin xyz="${d435_zero_depth_to_glass + d435_glass_to_front} ${-d435_cam_depth_py} 0" rpy="${M_PI/2} 0 ${M_PI/2}"/>
           <geometry>
-            <mesh filename="file://$(find hive_gazebo)/meshes/d435.dae" />
+            <mesh filename="file://$(find hive_gazebo)/meshes/intel_realsense/d435.dae" />
           </geometry>
         </xacro:if>

File: hive_gazebo/urdf/camera1/_usb_plug.urdf.xacro (robot description, xacro)
@@ -33,5 +33,5 @@
         <geometry>
           <!--box size="0.044850 0.008 0.0185" /-->
-          <mesh filename="file://$(find hive_gazebo)/meshes/plug.stl" />
+          <mesh filename="file://$(find hive_gazebo)/meshes/intel_realsense/plug.stl" />
         </geometry>
         <material name="plastic"/>
@@ -41,5 +41,5 @@
         <geometry>
           <!--box size="0.044850 0.008 0.0185" /-->
-          <mesh filename="file://$(find hive_gazebo)/meshes/plug_collision.stl" />
+          <mesh filename="file://$(find hive_gazebo)/meshes/intel_realsense/plug_collision.stl" />
         </geometry>
       </collision>

File: hive_gazebo/urdf/camera1/test_d435i_camera.urdf.xacro (robot description, xacro)
@@ -1,10 +1,11 @@
 <?xml version="1.0" ?>
-<robot name="realsense2_camera" xmlns:xacro="http://www.ros.org/wiki/xacro">
+<robot name="realsense2_camera"
+  xmlns:xacro="http://www.ros.org/wiki/xacro">
   <xacro:arg name="use_nominal_extrinsics" default="false" />
   <xacro:include filename="$(find hive_gazebo)/urdf/camera1/_d435i.urdf.xacro"/>
   <xacro:property name="M_PI" value="3.1415926535897931" />
-  <link name="ceiling_link" />
+  <link name="ceiling_link"/>
   <xacro:sensor_d435i parent="ceiling_link" use_nominal_extrinsics="$(arg use_nominal_extrinsics)">
-    <origin xyz="0 0 3.5" rpy="0 ${M_PI}/2 0"/>
+    <origin xyz="0 0 0" rpy="0 0 0"/>
   </xacro:sensor_d435i>
 </robot>
