Commit message: feat: add second camera urdf file.

File: hive_gazebo/urdf/camera2/test_d435i_camera.urdf.xacro (robot description, xacro)
@@ -3,10 +3,9 @@
   xmlns:xacro="http://www.ros.org/wiki/xacro">
   <xacro:arg name="use_nominal_extrinsics" default="false" />
-  <xacro:include filename="$(find hive_gazebo)/urdf/camera1/_d435i.urdf.xacro"/>
-  <xacro:include filename="$(find hive_gazebo)/urdf/camera1/camera1.gazebo"/>
+  <xacro:include filename="$(find hive_gazebo)/urdf/camera2/_d435i.urdf.xacro"/>
   <xacro:property name="M_PI" value="3.1415926535897931" />
   <link name="ceiling_link"/>
   <xacro:sensor_d435i parent="ceiling_link" use_nominal_extrinsics="$(arg use_nominal_extrinsics)">
-    <origin xyz="0.5 0 0" rpy="0 ${M_PI/2} 0"/>
+    <origin xyz="0 0.5 0" rpy="0 ${M_PI/2} 0"/>
   </xacro:sensor_d435i>
 </robot>
