Commit message: feat: divide .xacro and .gazebo file for multi robot build.

File: hive_gazebo/urdf/robot1/robot1.xacro (robot description, xacro)
@@ -1,8 +1,8 @@
 <?xml version="1.0" ?>
-<robot name="geunwoo" xmlns:xacro="http://www.ros.org/wiki/xacro">
-<xacro:include filename="$(find hive_gazebo)/urdf/materials.xacro" />
-<xacro:include filename="$(find hive_gazebo)/urdf/geunwoo.trans" />
-<xacro:include filename="$(find hive_gazebo)/urdf/geunwoo.gazebo" />
-<link name="base_link">
+<robot name="robot1" xmlns:xacro="http://www.ros.org/wiki/xacro">
+<xacro:include filename="$(find hive_gazebo)/urdf/robot1/robot1_materials.xacro"/>
+<xacro:include filename="$(find hive_gazebo)/urdf/robot1/robot1.trans"/>
+<xacro:include filename="$(find hive_gazebo)/urdf/robot1/robot1.gazebo"/>
+<link name="robot1_base_link">
   <inertial>
     <origin xyz="-0.10589890450472451 0.004101721807053668 0.2428453449181509" rpy="0 0 0"/>
@@ -25,5 +25,5 @@
   </collision>
 </link>
-<link name="left_wheel">
+<link name="robot1_left_wheel">
   <inertial>
     <origin xyz="2.6594023369474935e-07 -0.006200652298741449 -4.894162568547244e-09" rpy="0 0 0"/>
@@ -45,5 +45,5 @@
   </collision>
 </link>
-<link name="right_wheel">
+<link name="robot1_right_wheel">
   <inertial>
     <origin xyz="2.5883027950490597e-07 0.006201095560612602 -2.8975644106310483e-10" rpy="0 0 0"/>
@@ -65,5 +65,5 @@
   </collision>
 </link>
-<link name="right_caster">
+<link name="robot1_right_caster">
   <inertial>
     <origin xyz="-0.017519612985357313 2.0677910783639675e-07 -0.05240105157186727" rpy="0 0 0"/>
@@ -85,5 +85,5 @@
   </collision>
 </link>
-<link name="left_caster">
+<link name="robot1_left_caster">
   <inertial>
     <origin xyz="-0.017519612985357313 2.0677910747557426e-07 -0.05240105157186712" rpy="0 0 0"/>
@@ -105,26 +105,26 @@
   </collision>
 </link>
-<joint name="left_wheel_joint" type="continuous">
+<joint name="robot1_left_wheel_joint" type="continuous">
   <origin xyz="-1e-06 0.277578 0.0" rpy="0 0 0"/>
-  <parent link="base_link"/>
-  <child link="left_wheel"/>
+  <parent link="robot1_base_link"/>
+  <child link="robot1_left_wheel"/>
   <axis xyz="0.0 1.0 0.0"/>
 </joint>
-<joint name="right_wheel_joint" type="continuous">
+<joint name="robot1_right_wheel_joint" type="continuous">
   <origin xyz="-1e-06 -0.269222 0.0" rpy="0 0 0"/>
-  <parent link="base_link"/>
-  <child link="right_wheel"/>
+  <parent link="robot1_base_link"/>
+  <child link="robot1_right_wheel"/>
   <axis xyz="0.0 1.0 0.0"/>
 </joint>
-<joint name="right_caster_joint" type="continuous">
+<joint name="robot1_right_caster_joint" type="fixed">
   <origin xyz="-0.310001 -0.185822 0.043" rpy="0 0 0"/>
-  <parent link="base_link"/>
-  <child link="right_caster"/>
+  <parent link="robot1_base_link"/>
+  <child link="robot1_right_caster"/>
   <axis xyz="0.0 0.0 -1.0"/>
 </joint>
-<joint name="left_caster_joint" type="continuous">
+<joint name="robot1_left_caster_joint" type="fixed">
   <origin xyz="-0.310001 0.194178 0.043" rpy="0 0 0"/>
-  <parent link="base_link"/>
-  <child link="left_caster"/>
+  <parent link="robot1_base_link"/>
+  <child link="robot1_left_caster"/>
   <axis xyz="0.0 0.0 -1.0"/>
 </joint>

File: hive_gazebo/urdf/robot1/robot1_materials.xacro (robot description, xacro)
@@ -1,4 +1,4 @@
 <?xml version="1.0" ?>
-<robot name="geunwoo" xmlns:xacro="http://www.ros.org/wiki/xacro" >
+<robot name="robot1" xmlns:xacro="http://www.ros.org/wiki/xacro" >
 <material name="silver">
   <color rgba="0.700 0.700 0.700 1.000"/>

Commit message: refactor: split urdf files in intelrealsense and robots

File: hive_gazebo/urdf/robot1/robot1.xacro (robot description, xacro)
@@ -14,5 +14,5 @@
     <origin xyz="0 0 0" rpy="0 0 0"/>
     <geometry>
-      <mesh filename="file://$(find hive_gazebo)/meshes/base_link.stl" scale="0.001 0.001 0.001"/>
+      <mesh filename="file://$(find hive_gazebo)/meshes/robots/base_link.stl" scale="0.001 0.001 0.001"/>
     </geometry>
     <material name="silver"/>
@@ -21,5 +21,5 @@
     <origin xyz="0 0 0" rpy="0 0 0"/>
     <geometry>
-      <mesh filename="file://$(find hive_gazebo)/meshes/base_link.stl" scale="0.001 0.001 0.001"/>
+      <mesh filename="file://$(find hive_gazebo)/meshes/robots/base_link.stl" scale="0.001 0.001 0.001"/>
     </geometry>
   </collision>
@@ -34,5 +34,5 @@
     <origin xyz="1e-06 -0.277578 0.0" rpy="0 0 0"/>
     <geometry>
-      <mesh filename="file://$(find hive_gazebo)/meshes/left_wheel_1.stl" scale="0.001 0.001 0.001"/>
+      <mesh filename="file://$(find hive_gazebo)/meshes/robots/left_wheel_1.stl" scale="0.001 0.001 0.001"/>
     </geometry>
     <material name="silver"/>
@@ -41,5 +41,5 @@
     <origin xyz="1e-06 -0.277578 0.0" rpy="0 0 0"/>
     <geometry>
-      <mesh filename="file://$(find hive_gazebo)/meshes/left_wheel_1.stl" scale="0.001 0.001 0.001"/>
+      <mesh filename="file://$(find hive_gazebo)/meshes/robots/left_wheel_1.stl" scale="0.001 0.001 0.001"/>
     </geometry>
   </collision>
@@ -54,5 +54,5 @@
     <origin xyz="1e-06 0.269222 0.0" rpy="0 0 0"/>
     <geometry>
-      <mesh filename="file://$(find hive_gazebo)/meshes/right_wheel_1.stl" scale="0.001 0.001 0.001"/>
+      <mesh filename="file://$(find hive_gazebo)/meshes/robots/right_wheel_1.stl" scale="0.001 0.001 0.001"/>
     </geometry>
     <material name="silver"/>
@@ -61,5 +61,5 @@
     <origin xyz="1e-06 0.269222 0.0" rpy="0 0 0"/>
     <geometry>
-      <mesh filename="file://$(find hive_gazebo)/meshes/right_wheel_1.stl" scale="0.001 0.001 0.001"/>
+      <mesh filename="file://$(find hive_gazebo)/meshes/robots/right_wheel_1.stl" scale="0.001 0.001 0.001"/>
     </geometry>
   </collision>
@@ -74,5 +74,5 @@
     <origin xyz="0.310001 0.185822 -0.043" rpy="0 0 0"/>
     <geometry>
-      <mesh filename="file://$(find hive_gazebo)/meshes/right_caster_1.stl" scale="0.001 0.001 0.001"/>
+      <mesh filename="file://$(find hive_gazebo)/meshes/robots/right_caster_1.stl" scale="0.001 0.001 0.001"/>
     </geometry>
     <material name="silver"/>
@@ -81,5 +81,5 @@
     <origin xyz="0.310001 0.185822 -0.043" rpy="0 0 0"/>
     <geometry>
-      <mesh filename="file://$(find hive_gazebo)/meshes/right_caster_1.stl" scale="0.001 0.001 0.001"/>
+      <mesh filename="file://$(find hive_gazebo)/meshes/robots/right_caster_1.stl" scale="0.001 0.001 0.001"/>
     </geometry>
   </collision>
@@ -94,5 +94,5 @@
     <origin xyz="0.310001 -0.194178 -0.043" rpy="0 0 0"/>
     <geometry>
-      <mesh filename="file://$(find hive_gazebo)/meshes/left_caster_1.stl" scale="0.001 0.001 0.001"/>
+      <mesh filename="file://$(find hive_gazebo)/meshes/robots/left_caster_1.stl" scale="0.001 0.001 0.001"/>
     </geometry>
     <material name="silver"/>
@@ -101,5 +101,5 @@
     <origin xyz="0.310001 -0.194178 -0.043" rpy="0 0 0"/>
     <geometry>
-      <mesh filename="file://$(find hive_gazebo)/meshes/left_caster_1.stl" scale="0.001 0.001 0.001"/>
+      <mesh filename="file://$(find hive_gazebo)/meshes/robots/left_caster_1.stl" scale="0.001 0.001 0.001"/>
     </geometry>
   </collision>

File: hive_gazebo/urdf/robot2/robot2.xacro (robot description, xacro)
@@ -14,5 +14,5 @@
     <origin xyz="0 0 0" rpy="0 0 0"/>
     <geometry>
-      <mesh filename="file://$(find hive_gazebo)/meshes/base_link.stl" scale="0.001 0.001 0.001"/>
+      <mesh filename="file://$(find hive_gazebo)/meshes/robots/base_link.stl" scale="0.001 0.001 0.001"/>
     </geometry>
     <material name="red"/>
@@ -21,5 +21,5 @@
     <origin xyz="0 0 0" rpy="0 0 0"/>
     <geometry>
-      <mesh filename="file://$(find hive_gazebo)/meshes/base_link.stl" scale="0.001 0.001 0.001"/>
+      <mesh filename="file://$(find hive_gazebo)/meshes/robots/base_link.stl" scale="0.001 0.001 0.001"/>
     </geometry>
   </collision>
@@ -34,5 +34,5 @@
     <origin xyz="1e-06 -0.277578 0.0" rpy="0 0 0"/>
     <geometry>
-      <mesh filename="file://$(find hive_gazebo)/meshes/left_wheel_1.stl" scale="0.001 0.001 0.001"/>
+      <mesh filename="file://$(find hive_gazebo)/meshes/robots/left_wheel_1.stl" scale="0.001 0.001 0.001"/>
     </geometry>
     <material name="red"/>
@@ -41,5 +41,5 @@
     <origin xyz="1e-06 -0.277578 0.0" rpy="0 0 0"/>
     <geometry>
-      <mesh filename="file://$(find hive_gazebo)/meshes/left_wheel_1.stl" scale="0.001 0.001 0.001"/>
+      <mesh filename="file://$(find hive_gazebo)/meshes/robots/left_wheel_1.stl" scale="0.001 0.001 0.001"/>
     </geometry>
   </collision>
@@ -54,5 +54,5 @@
     <origin xyz="1e-06 0.269222 0.0" rpy="0 0 0"/>
     <geometry>
-      <mesh filename="file://$(find hive_gazebo)/meshes/right_wheel_1.stl" scale="0.001 0.001 0.001"/>
+      <mesh filename="file://$(find hive_gazebo)/meshes/robots/right_wheel_1.stl" scale="0.001 0.001 0.001"/>
     </geometry>
     <material name="red"/>
@@ -61,5 +61,5 @@
     <origin xyz="1e-06 0.269222 0.0" rpy="0 0 0"/>
     <geometry>
-      <mesh filename="file://$(find hive_gazebo)/meshes/right_wheel_1.stl" scale="0.001 0.001 0.001"/>
+      <mesh filename="file://$(find hive_gazebo)/meshes/robots/right_wheel_1.stl" scale="0.001 0.001 0.001"/>
     </geometry>
   </collision>
@@ -74,5 +74,5 @@
     <origin xyz="0.310001 0.185822 -0.043" rpy="0 0 0"/>
     <geometry>
-      <mesh filename="file://$(find hive_gazebo)/meshes/right_caster_1.stl" scale="0.001 0.001 0.001"/>
+      <mesh filename="file://$(find hive_gazebo)/meshes/robots/right_caster_1.stl" scale="0.001 0.001 0.001"/>
     </geometry>
     <material name="red"/>
@@ -81,5 +81,5 @@
     <origin xyz="0.310001 0.185822 -0.043" rpy="0 0 0"/>
     <geometry>
-      <mesh filename="file://$(find hive_gazebo)/meshes/right_caster_1.stl" scale="0.001 0.001 0.001"/>
+      <mesh filename="file://$(find hive_gazebo)/meshes/robots/right_caster_1.stl" scale="0.001 0.001 0.001"/>
     </geometry>
   </collision>
@@ -94,5 +94,5 @@
     <origin xyz="0.310001 -0.194178 -0.043" rpy="0 0 0"/>
     <geometry>
-      <mesh filename="file://$(find hive_gazebo)/meshes/left_caster_1.stl" scale="0.001 0.001 0.001"/>
+      <mesh filename="file://$(find hive_gazebo)/meshes/robots/left_caster_1.stl" scale="0.001 0.001 0.001"/>
     </geometry>
     <material name="red"/>
@@ -101,5 +101,5 @@
     <origin xyz="0.310001 -0.194178 -0.043" rpy="0 0 0"/>
     <geometry>
-      <mesh filename="file://$(find hive_gazebo)/meshes/left_caster_1.stl" scale="0.001 0.001 0.001"/>
+      <mesh filename="file://$(find hive_gazebo)/meshes/robots/left_caster_1.stl" scale="0.001 0.001 0.001"/>
     </geometry>
   </collision>

File: hive_gazebo/urdf/robot3/robot3.xacro (robot description, xacro)
@@ -14,5 +14,5 @@
     <origin xyz="0 0 0" rpy="0 0 0"/>
     <geometry>
-      <mesh filename="file://$(find hive_gazebo)/meshes/base_link.stl" scale="0.001 0.001 0.001"/>
+      <mesh filename="file://$(find hive_gazebo)/meshes/robots/base_link.stl" scale="0.001 0.001 0.001"/>
     </geometry>
     <material name="green"/>
@@ -21,5 +21,5 @@
     <origin xyz="0 0 0" rpy="0 0 0"/>
     <geometry>
-      <mesh filename="file://$(find hive_gazebo)/meshes/base_link.stl" scale="0.001 0.001 0.001"/>
+      <mesh filename="file://$(find hive_gazebo)/meshes/robots/base_link.stl" scale="0.001 0.001 0.001"/>
     </geometry>
   </collision>
@@ -34,5 +34,5 @@
     <origin xyz="1e-06 -0.277578 0.0" rpy="0 0 0"/>
     <geometry>
-      <mesh filename="file://$(find hive_gazebo)/meshes/left_wheel_1.stl" scale="0.001 0.001 0.001"/>
+      <mesh filename="file://$(find hive_gazebo)/meshes/robots/left_wheel_1.stl" scale="0.001 0.001 0.001"/>
     </geometry>
     <material name="green"/>
@@ -41,5 +41,5 @@
     <origin xyz="1e-06 -0.277578 0.0" rpy="0 0 0"/>
     <geometry>
-      <mesh filename="file://$(find hive_gazebo)/meshes/left_wheel_1.stl" scale="0.001 0.001 0.001"/>
+      <mesh filename="file://$(find hive_gazebo)/meshes/robots/left_wheel_1.stl" scale="0.001 0.001 0.001"/>
     </geometry>
   </collision>
@@ -54,5 +54,5 @@
     <origin xyz="1e-06 0.269222 0.0" rpy="0 0 0"/>
     <geometry>
-      <mesh filename="file://$(find hive_gazebo)/meshes/right_wheel_1.stl" scale="0.001 0.001 0.001"/>
+      <mesh filename="file://$(find hive_gazebo)/meshes/robots/right_wheel_1.stl" scale="0.001 0.001 0.001"/>
     </geometry>
     <material name="green"/>
@@ -61,5 +61,5 @@
     <origin xyz="1e-06 0.269222 0.0" rpy="0 0 0"/>
     <geometry>
-      <mesh filename="file://$(find hive_gazebo)/meshes/right_wheel_1.stl" scale="0.001 0.001 0.001"/>
+      <mesh filename="file://$(find hive_gazebo)/meshes/robots/right_wheel_1.stl" scale="0.001 0.001 0.001"/>
     </geometry>
   </collision>
@@ -74,5 +74,5 @@
     <origin xyz="0.310001 0.185822 -0.043" rpy="0 0 0"/>
     <geometry>
-      <mesh filename="file://$(find hive_gazebo)/meshes/right_caster_1.stl" scale="0.001 0.001 0.001"/>
+      <mesh filename="file://$(find hive_gazebo)/meshes/robots/right_caster_1.stl" scale="0.001 0.001 0.001"/>
     </geometry>
     <material name="green"/>
@@ -81,5 +81,5 @@
     <origin xyz="0.310001 0.185822 -0.043" rpy="0 0 0"/>
     <geometry>
-      <mesh filename="file://$(find hive_gazebo)/meshes/right_caster_1.stl" scale="0.001 0.001 0.001"/>
+      <mesh filename="file://$(find hive_gazebo)/meshes/robots/right_caster_1.stl" scale="0.001 0.001 0.001"/>
     </geometry>
   </collision>
@@ -94,5 +94,5 @@
     <origin xyz="0.310001 -0.194178 -0.043" rpy="0 0 0"/>
     <geometry>
-      <mesh filename="file://$(find hive_gazebo)/meshes/left_caster_1.stl" scale="0.001 0.001 0.001"/>
+      <mesh filename="file://$(find hive_gazebo)/meshes/robots/left_caster_1.stl" scale="0.001 0.001 0.001"/>
     </geometry>
     <material name="green"/>
@@ -101,5 +101,5 @@
     <origin xyz="0.310001 -0.194178 -0.043" rpy="0 0 0"/>
     <geometry>
-      <mesh filename="file://$(find hive_gazebo)/meshes/left_caster_1.stl" scale="0.001 0.001 0.001"/>
+      <mesh filename="file://$(find hive_gazebo)/meshes/robots/left_caster_1.stl" scale="0.001 0.001 0.001"/>
     </geometry>
   </collision>

Commit message: feat: modify urdf and add lidar

File: hive_gazebo/urdf/robot1/robot1.xacro (robot description, xacro)
@@ -6,8 +6,7 @@
 <link name="robot1_base_link">
   <inertial>
-    <origin xyz="-0.10589890450472451 0.004101721807053668 0.2428453449181509" rpy="0 0 0"/>
-    <!-- <mass value="97.68742911120015"/> -->
+    <origin xyz="-0.10420283159261519 -6.650792304374791e-05 0.2749529701185766" rpy="0 0 0"/>
     <mass value="40.0"/>
-    <inertia ixx="5.633563" iyy="4.887417" izz="5.433869" ixy="0.000389" iyz="-0.000239" ixz="0.200866"/>
+    <inertia ixx="6.809657" iyy="6.121132" izz="6.33059" ixy="0.000377" iyz="-0.000479" ixz="0.18348"/>
   </inertial>
   <visual>
@@ -105,6 +104,26 @@
   </collision>
 </link>
+<link name="robot1_lidar_link">
+  <inertial>
+    <origin xyz="-0.0005135302448306955 -0.0001199429580434408 0.02218628196103728" rpy="0 0 0"/>
+    <mass value="1.4419128562477859"/>
+    <inertia ixx="0.000731" iyy="0.000735" izz="0.000958" ixy="3e-06" iyz="2e-06" ixz="8e-06"/>
+  </inertial>
+  <visual>
+    <origin xyz="0.12 0.0 -0.395" rpy="0 0 0"/>
+    <geometry>
+      <mesh filename="file://$(find hive_gazebo)/meshes/robots/lidar_link_1.stl" scale="0.001 0.001 0.001"/>
+    </geometry>
+    <material name="silver"/>
+  </visual>
+  <collision>
+    <origin xyz="0.12 0.0 -0.395" rpy="0 0 0"/>
+    <geometry>
+      <mesh filename="file://$(find hive_gazebo)/meshes/robots/lidar_link_1.stl" scale="0.001 0.001 0.001"/>
+    </geometry>
+  </collision>
+</link>
 <joint name="robot1_left_wheel_joint" type="continuous">
-  <origin xyz="-1e-06 0.277578 0.0" rpy="0 0 0"/>
+  <origin xyz="-1e-06 0.2734 0.0" rpy="0 0 0"/>
   <parent link="robot1_base_link"/>
   <child link="robot1_left_wheel"/>
@@ -112,5 +131,5 @@
 </joint>
 <joint name="robot1_right_wheel_joint" type="continuous">
-  <origin xyz="-1e-06 -0.269222 0.0" rpy="0 0 0"/>
+  <origin xyz="-1e-06 -0.2734 0.0" rpy="0 0 0"/>
   <parent link="robot1_base_link"/>
   <child link="robot1_right_wheel"/>
@@ -118,5 +137,5 @@
 </joint>
 <joint name="robot1_right_caster_joint" type="fixed">
-  <origin xyz="-0.310001 -0.185822 0.043" rpy="0 0 0"/>
+  <origin xyz="-0.31 -0.19 0.043" rpy="0 0 0"/>
   <parent link="robot1_base_link"/>
   <child link="robot1_right_caster"/>
@@ -124,8 +143,14 @@
 </joint>
 <joint name="robot1_left_caster_joint" type="fixed">
-  <origin xyz="-0.310001 0.194178 0.043" rpy="0 0 0"/>
+  <origin xyz="-0.31 0.19 0.043" rpy="0 0 0"/>
   <parent link="robot1_base_link"/>
   <child link="robot1_left_caster"/>
   <axis xyz="0.0 0.0 -1.0"/>
 </joint>
+<joint name="robot1_lidar_joint" type="fixed">
+  <origin xyz="-0.12 0.0 0.405" rpy="0 0 0"/>
+  <parent link="robot1_base_link"/>
+  <child link="robot1_lidar_link"/>
+  <axis xyz="-0.0 -0.0 1.0"/>
+</joint>
 </robot>

File: hive_gazebo/urdf/robot2/robot2.xacro (robot description, xacro)
@@ -6,8 +6,7 @@
 <link name="robot2_base_link">
   <inertial>
-    <origin xyz="-0.10589890450472451 0.004101721807053668 0.2428453449181509" rpy="0 0 0"/>
-    <!-- <mass value="97.68742911120015"/> -->
+    <origin xyz="-0.10420283159261519 -6.650792304374791e-05 0.2749529701185766" rpy="0 0 0"/>
     <mass value="40.0"/>
-    <inertia ixx="5.633563" iyy="4.887417" izz="5.433869" ixy="0.000389" iyz="-0.000239" ixz="0.200866"/>
+    <inertia ixx="6.809657" iyy="6.121132" izz="6.33059" ixy="0.000377" iyz="-0.000479" ixz="0.18348"/>
   </inertial>
   <visual>
@@ -105,6 +104,26 @@
   </collision>
 </link>
+<link name="robot2_lidar_link">
+  <inertial>
+    <origin xyz="-0.0005135302448306955 -0.0001199429580434408 0.02218628196103728" rpy="0 0 0"/>
+    <mass value="1.4419128562477859"/>
+    <inertia ixx="0.000731" iyy="0.000735" izz="0.000958" ixy="3e-06" iyz="2e-06" ixz="8e-06"/>
+  </inertial>
+  <visual>
+    <origin xyz="0.12 0.0 -0.395" rpy="0 0 0"/>
+    <geometry>
+      <mesh filename="file://$(find hive_gazebo)/meshes/robots/lidar_link_1.stl" scale="0.001 0.001 0.001"/>
+    </geometry>
+    <material name="red"/>
+  </visual>
+  <collision>
+    <origin xyz="0.12 0.0 -0.395" rpy="0 0 0"/>
+    <geometry>
+      <mesh filename="file://$(find hive_gazebo)/meshes/robots/lidar_link_1.stl" scale="0.001 0.001 0.001"/>
+    </geometry>
+  </collision>
+</link>
 <joint name="robot2_left_wheel_joint" type="continuous">
-  <origin xyz="-1e-06 0.277578 0.0" rpy="0 0 0"/>
+  <origin xyz="-1e-06 0.2734 0.0" rpy="0 0 0"/>
   <parent link="robot2_base_link"/>
   <child link="robot2_left_wheel"/>
@@ -112,5 +131,5 @@
 </joint>
 <joint name="robot2_right_wheel_joint" type="continuous">
-  <origin xyz="-1e-06 -0.269222 0.0" rpy="0 0 0"/>
+  <origin xyz="-1e-06 -0.2734 0.0" rpy="0 0 0"/>
   <parent link="robot2_base_link"/>
   <child link="robot2_right_wheel"/>
@@ -118,5 +137,5 @@
 </joint>
 <joint name="robot2_right_caster_joint" type="fixed">
-  <origin xyz="-0.310001 -0.185822 0.043" rpy="0 0 0"/>
+  <origin xyz="-0.31 -0.19 0.043" rpy="0 0 0"/>
   <parent link="robot2_base_link"/>
   <child link="robot2_right_caster"/>
@@ -124,8 +143,14 @@
 </joint>
 <joint name="robot2_left_caster_joint" type="fixed">
-  <origin xyz="-0.310001 0.194178 0.043" rpy="0 0 0"/>
+  <origin xyz="-0.31 0.19 0.043" rpy="0 0 0"/>
   <parent link="robot2_base_link"/>
   <child link="robot2_left_caster"/>
   <axis xyz="0.0 0.0 -1.0"/>
 </joint>
+<joint name="robot2_lidar_joint" type="fixed">
+  <origin xyz="-0.12 0.0 0.405" rpy="0 0 0"/>
+  <parent link="robot2_base_link"/>
+  <child link="robot2_lidar_link"/>
+  <axis xyz="-0.0 -0.0 1.0"/>
+</joint>
 </robot>

File: hive_gazebo/urdf/robot3/robot3.xacro (robot description, xacro)
@@ -6,8 +6,7 @@
 <link name="robot3_base_link">
   <inertial>
-    <origin xyz="-0.10589890450472451 0.004101721807053668 0.2428453449181509" rpy="0 0 0"/>
-    <!-- <mass value="97.68742911120015"/> -->
+    <origin xyz="-0.10420283159261519 -6.650792304374791e-05 0.2749529701185766" rpy="0 0 0"/>
     <mass value="40.0"/>
-    <inertia ixx="5.633563" iyy="4.887417" izz="5.433869" ixy="0.000389" iyz="-0.000239" ixz="0.200866"/>
+    <inertia ixx="6.809657" iyy="6.121132" izz="6.33059" ixy="0.000377" iyz="-0.000479" ixz="0.18348"/>
   </inertial>
   <visual>
@@ -105,6 +104,26 @@
   </collision>
 </link>
+<link name="robot3_lidar_link">
+  <inertial>
+    <origin xyz="-0.0005135302448306955 -0.0001199429580434408 0.02218628196103728" rpy="0 0 0"/>
+    <mass value="1.4419128562477859"/>
+    <inertia ixx="0.000731" iyy="0.000735" izz="0.000958" ixy="3e-06" iyz="2e-06" ixz="8e-06"/>
+  </inertial>
+  <visual>
+    <origin xyz="0.12 0.0 -0.395" rpy="0 0 0"/>
+    <geometry>
+      <mesh filename="file://$(find hive_gazebo)/meshes/robots/lidar_link_1.stl" scale="0.001 0.001 0.001"/>
+    </geometry>
+    <material name="green"/>
+  </visual>
+  <collision>
+    <origin xyz="0.12 0.0 -0.395" rpy="0 0 0"/>
+    <geometry>
+      <mesh filename="file://$(find hive_gazebo)/meshes/robots/lidar_link_1.stl" scale="0.001 0.001 0.001"/>
+    </geometry>
+  </collision>
+</link>
 <joint name="robot3_left_wheel_joint" type="continuous">
-  <origin xyz="-1e-06 0.277578 0.0" rpy="0 0 0"/>
+  <origin xyz="-1e-06 0.2734 0.0" rpy="0 0 0"/>
   <parent link="robot3_base_link"/>
   <child link="robot3_left_wheel"/>
@@ -112,5 +131,5 @@
 </joint>
 <joint name="robot3_right_wheel_joint" type="continuous">
-  <origin xyz="-1e-06 -0.269222 0.0" rpy="0 0 0"/>
+  <origin xyz="-1e-06 -0.2734 0.0" rpy="0 0 0"/>
   <parent link="robot3_base_link"/>
   <child link="robot3_right_wheel"/>
@@ -118,5 +137,5 @@
 </joint>
 <joint name="robot3_right_caster_joint" type="fixed">
-  <origin xyz="-0.310001 -0.185822 0.043" rpy="0 0 0"/>
+  <origin xyz="-0.31 -0.19 0.043" rpy="0 0 0"/>
   <parent link="robot3_base_link"/>
   <child link="robot3_right_caster"/>
@@ -124,8 +143,14 @@
 </joint>
 <joint name="robot3_left_caster_joint" type="fixed">
-  <origin xyz="-0.310001 0.194178 0.043" rpy="0 0 0"/>
+  <origin xyz="-0.31 0.19 0.043" rpy="0 0 0"/>
   <parent link="robot3_base_link"/>
   <child link="robot3_left_caster"/>
   <axis xyz="0.0 0.0 -1.0"/>
 </joint>
+<joint name="robot3_lidar_joint" type="fixed">
+  <origin xyz="-0.12 0.0 0.405" rpy="0 0 0"/>
+  <parent link="robot3_base_link"/>
+  <child link="robot3_lidar_link"/>
+  <axis xyz="-0.0 -0.0 1.0"/>
+</joint>
 </robot>
