Commit message: change robot color same to real hardware

File: hive_gazebo/urdf/robot1/robot1.xacro (robot description, xacro)
@@ -15,5 +15,5 @@
       <mesh filename="file://$(find hive_gazebo)/meshes/robots/base_link.stl" scale="0.001 0.001 0.001"/>
     </geometry>
-    <material name="silver"/>
+    <material name="blue"/>
   </visual>
   <collision>
@@ -35,5 +35,5 @@
       <mesh filename="file://$(find hive_gazebo)/meshes/robots/left_wheel_1.stl" scale="0.001 0.001 0.001"/>
     </geometry>
-    <material name="silver"/>
+    <material name="blue"/>
   </visual>
   <collision>
@@ -55,5 +55,5 @@
       <mesh filename="file://$(find hive_gazebo)/meshes/robots/right_wheel_1.stl" scale="0.001 0.001 0.001"/>
     </geometry>
-    <material name="silver"/>
+    <material name="blue"/>
   </visual>
   <collision>
@@ -75,5 +75,5 @@
       <mesh filename="file://$(find hive_gazebo)/meshes/robots/right_caster_1.stl" scale="0.001 0.001 0.001"/>
     </geometry>
-    <material name="silver"/>
+    <material name="blue"/>
   </visual>
   <collision>
@@ -95,5 +95,5 @@
       <mesh filename="file://$(find hive_gazebo)/meshes/robots/left_caster_1.stl" scale="0.001 0.001 0.001"/>
     </geometry>
-    <material name="silver"/>
+    <material name="blue"/>
   </visual>
   <collision>
@@ -115,5 +115,5 @@
       <mesh filename="file://$(find hive_gazebo)/meshes/robots/lidar_link_1.stl" scale="0.001 0.001 0.001"/>
     </geometry>
-    <material name="silver"/>
+    <material name="blue"/>
   </visual>
   <collision>

File: hive_gazebo/urdf/robot1/robot1_materials.xacro (robot description, xacro)
@@ -1,6 +1,6 @@
 <?xml version="1.0" ?>
 <robot name="robot1" xmlns:xacro="http://www.ros.org/wiki/xacro" >
-<material name="silver">
-  <color rgba="0.700 0.700 0.700 1.000"/>
+<material name="blue">
+  <color rgba="0.000 0.000 0.700 1.000"/>
 </material>
 </robot>

File: hive_gazebo/urdf/robot2/robot2.xacro (robot description, xacro)
@@ -15,5 +15,5 @@
       <mesh filename="file://$(find hive_gazebo)/meshes/robots/base_link.stl" scale="0.001 0.001 0.001"/>
     </geometry>
-    <material name="red"/>
+    <material name="blue"/>
   </visual>
   <collision>
@@ -35,5 +35,5 @@
       <mesh filename="file://$(find hive_gazebo)/meshes/robots/left_wheel_1.stl" scale="0.001 0.001 0.001"/>
     </geometry>
-    <material name="red"/>
+    <material name="blue"/>
   </visual>
   <collision>
@@ -55,5 +55,5 @@
       <mesh filename="file://$(find hive_gazebo)/meshes/robots/right_wheel_1.stl" scale="0.001 0.001 0.001"/>
     </geometry>
-    <material name="red"/>
+    <material name="blue"/>
   </visual>
   <collision>
@@ -75,5 +75,5 @@
       <mesh filename="file://$(find hive_gazebo)/meshes/robots/right_caster_1.stl" scale="0.001 0.001 0.001"/>
     </geometry>
-    <material name="red"/>
+    <material name="blue"/>
   </visual>
   <collision>
@@ -95,5 +95,5 @@
       <mesh filename="file://$(find hive_gazebo)/meshes/robots/left_caster_1.stl" scale="0.001 0.001 0.001"/>
     </geometry>
-    <material name="red"/>
+    <material name="blue"/>
   </visual>
   <collision>
@@ -115,5 +115,5 @@
       <mesh filename="file://$(find hive_gazebo)/meshes/robots/lidar_link_1.stl" scale="0.001 0.001 0.001"/>
     </geometry>
-    <material name="red"/>
+    <material name="blue"/>
   </visual>
   <collision>

File: hive_gazebo/urdf/robot2/robot2_materials.xacro (robot description, xacro)
@@ -1,6 +1,6 @@
 <?xml version="1.0" ?>
 <robot name="robot2" xmlns:xacro="http://www.ros.org/wiki/xacro" >
-<material name="red">
-  <color rgba="0.700 0.000 0.000 1.000"/>
+<material name="blue">
+  <color rgba="0.000 0.000 0.700 1.000"/>
 </material>
 </robot>

File: hive_gazebo/urdf/robot3/robot3.xacro (robot description, xacro)
@@ -15,5 +15,5 @@
       <mesh filename="file://$(find hive_gazebo)/meshes/robots/base_link.stl" scale="0.001 0.001 0.001"/>
     </geometry>
-    <material name="green"/>
+    <material name="blue"/>
   </visual>
   <collision>
@@ -35,5 +35,5 @@
       <mesh filename="file://$(find hive_gazebo)/meshes/robots/left_wheel_1.stl" scale="0.001 0.001 0.001"/>
     </geometry>
-    <material name="green"/>
+    <material name="blue"/>
   </visual>
   <collision>
@@ -55,5 +55,5 @@
       <mesh filename="file://$(find hive_gazebo)/meshes/robots/right_wheel_1.stl" scale="0.001 0.001 0.001"/>
     </geometry>
-    <material name="green"/>
+    <material name="blue"/>
   </visual>
   <collision>
@@ -75,5 +75,5 @@
       <mesh filename="file://$(find hive_gazebo)/meshes/robots/right_caster_1.stl" scale="0.001 0.001 0.001"/>
     </geometry>
-    <material name="green"/>
+    <material name="blue"/>
   </visual>
   <collision>
@@ -95,5 +95,5 @@
       <mesh filename="file://$(find hive_gazebo)/meshes/robots/left_caster_1.stl" scale="0.001 0.001 0.001"/>
     </geometry>
-    <material name="green"/>
+    <material name="blue"/>
   </visual>
   <collision>
@@ -115,5 +115,5 @@
       <mesh filename="file://$(find hive_gazebo)/meshes/robots/lidar_link_1.stl" scale="0.001 0.001 0.001"/>
     </geometry>
-    <material name="green"/>
+    <material name="blue"/>
   </visual>
   <collision>

File: hive_gazebo/urdf/robot3/robot3_materials.xacro (robot description, xacro)
@@ -1,6 +1,6 @@
 <?xml version="1.0" ?>
 <robot name="robot3" xmlns:xacro="http://www.ros.org/wiki/xacro" >
-<material name="green">
-  <color rgba="0.000 0.500 0.000 1.000"/>
+<material name="blue">
+  <color rgba="0.000 0.000 0.700 1.000"/>
 </material>
 </robot>

Commit message: feat: add imu plugins.

File: hive_gazebo/urdf/robot1/robot1.xacro (robot description, xacro)
@@ -124,4 +124,10 @@
   </collision>
 </link>
+<link name="robot1_imu_link"/>
+<joint name="robot1_imu_joint" type="fixed">
+  <origin xyz="-0.12 0 0.5" rpy="0 0 0"/>
+  <parent link="robot1_base_link"/>
+  <child link="robot1_imu_link"/>
+</joint>
 <joint name="robot1_left_wheel_joint" type="continuous">
   <origin xyz="-1e-06 0.2734 0.0" rpy="0 0 0"/>

File: hive_gazebo/urdf/robot2/robot2.xacro (robot description, xacro)
@@ -1,156 +1,163 @@
 <?xml version="1.0" ?>
-<robot name="robot2" xmlns:xacro="http://www.ros.org/wiki/xacro">
-<xacro:include filename="$(find hive_gazebo)/urdf/robot2/robot2_materials.xacro"/>
-<xacro:include filename="$(find hive_gazebo)/urdf/robot2/robot2.trans"/>
-<xacro:include filename="$(find hive_gazebo)/urdf/robot2/robot2.gazebo"/>
-<link name="robot2_base_link">
-  <inertial>
-    <origin xyz="-0.10420283159261519 -6.650792304374791e-05 0.2749529701185766" rpy="0 0 0"/>
-    <mass value="40.0"/>
-    <inertia ixx="6.809657" iyy="6.121132" izz="6.33059" ixy="0.000377" iyz="-0.000479" ixz="0.18348"/>
-  </inertial>
-  <visual>
-    <origin xyz="0 0 0" rpy="0 0 0"/>
-    <geometry>
-      <mesh filename="file://$(find hive_gazebo)/meshes/robots/base_link.stl" scale="0.001 0.001 0.001"/>
-    </geometry>
-    <material name="blue"/>
-  </visual>
-  <collision>
-    <origin xyz="0 0 0" rpy="0 0 0"/>
-    <geometry>
-      <mesh filename="file://$(find hive_gazebo)/meshes/robots/base_link.stl" scale="0.001 0.001 0.001"/>
-    </geometry>
-  </collision>
-</link>
-<link name="robot2_left_wheel">
-  <inertial>
-    <origin xyz="2.6594023369474935e-07 -0.006200652298741449 -4.894162568547244e-09" rpy="0 0 0"/>
-    <mass value="1.3260899817774452"/>
-    <inertia ixx="0.001415" iyy="0.002676" izz="0.001415" ixy="-0.0" iyz="0.0" ixz="0.0"/>
-  </inertial>
-  <visual>
-    <origin xyz="1e-06 -0.277578 0.0" rpy="0 0 0"/>
-    <geometry>
-      <mesh filename="file://$(find hive_gazebo)/meshes/robots/left_wheel_1.stl" scale="0.001 0.001 0.001"/>
-    </geometry>
-    <material name="blue"/>
-  </visual>
-  <collision>
-    <origin xyz="1e-06 -0.277578 0.0" rpy="0 0 0"/>
-    <geometry>
-      <mesh filename="file://$(find hive_gazebo)/meshes/robots/left_wheel_1.stl" scale="0.001 0.001 0.001"/>
-    </geometry>
-  </collision>
-</link>
-<link name="robot2_right_wheel">
-  <inertial>
-    <origin xyz="2.5883027950490597e-07 0.006201095560612602 -2.8975644106310483e-10" rpy="0 0 0"/>
-    <mass value="1.3260894987915728"/>
-    <inertia ixx="0.001415" iyy="0.002676" izz="0.001415" ixy="-0.0" iyz="0.0" ixz="-0.0"/>
-  </inertial>
-  <visual>
-    <origin xyz="1e-06 0.269222 0.0" rpy="0 0 0"/>
-    <geometry>
-      <mesh filename="file://$(find hive_gazebo)/meshes/robots/right_wheel_1.stl" scale="0.001 0.001 0.001"/>
-    </geometry>
-    <material name="blue"/>
-  </visual>
-  <collision>
-    <origin xyz="1e-06 0.269222 0.0" rpy="0 0 0"/>
-    <geometry>
-      <mesh filename="file://$(find hive_gazebo)/meshes/robots/right_wheel_1.stl" scale="0.001 0.001 0.001"/>
-    </geometry>
-  </collision>
-</link>
-<link name="robot2_right_caster">
-  <inertial>
-    <origin xyz="-0.017519612985357313 2.0677910783639675e-07 -0.05240105157186727" rpy="0 0 0"/>
-    <mass value="1.6117875662608887"/>
-    <inertia ixx="0.001424" iyy="0.001841" izz="0.000923" ixy="-0.0" iyz="-0.0" ixz="-0.000298"/>
-  </inertial>
-  <visual>
-    <origin xyz="0.310001 0.185822 -0.043" rpy="0 0 0"/>
-    <geometry>
-      <mesh filename="file://$(find hive_gazebo)/meshes/robots/right_caster_1.stl" scale="0.001 0.001 0.001"/>
-    </geometry>
-    <material name="blue"/>
-  </visual>
-  <collision>
-    <origin xyz="0.310001 0.185822 -0.043" rpy="0 0 0"/>
-    <geometry>
-      <mesh filename="file://$(find hive_gazebo)/meshes/robots/right_caster_1.stl" scale="0.001 0.001 0.001"/>
-    </geometry>
-  </collision>
-</link>
-<link name="robot2_left_caster">
-  <inertial>
-    <origin xyz="-0.017519612985357313 2.0677910747557426e-07 -0.05240105157186712" rpy="0 0 0"/>
-    <mass value="1.6117875662608847"/>
-    <inertia ixx="0.001424" iyy="0.001841" izz="0.000923" ixy="-0.0" iyz="-0.0" ixz="-0.000298"/>
-  </inertial>
-  <visual>
-    <origin xyz="0.310001 -0.194178 -0.043" rpy="0 0 0"/>
-    <geometry>
-      <mesh filename="file://$(find hive_gazebo)/meshes/robots/left_caster_1.stl" scale="0.001 0.001 0.001"/>
-    </geometry>
-    <material name="blue"/>
-  </visual>
-  <collision>
-    <origin xyz="0.310001 -0.194178 -0.043" rpy="0 0 0"/>
-    <geometry>
-      <mesh filename="file://$(find hive_gazebo)/meshes/robots/left_caster_1.stl" scale="0.001 0.001 0.001"/>
-    </geometry>
-  </collision>
-</link>
-<link name="robot2_lidar_link">
-  <inertial>
-    <origin xyz="-0.0005135302448306955 -0.0001199429580434408 0.02218628196103728" rpy="0 0 0"/>
-    <mass value="1.4419128562477859"/>
-    <inertia ixx="0.000731" iyy="0.000735" izz="0.000958" ixy="3e-06" iyz="2e-06" ixz="8e-06"/>
-  </inertial>
-  <visual>
-    <origin xyz="0.12 0.0 -0.395" rpy="0 0 0"/>
-    <geometry>
-      <mesh filename="file://$(find hive_gazebo)/meshes/robots/lidar_link_1.stl" scale="0.001 0.001 0.001"/>
-    </geometry>
-    <material name="blue"/>
-  </visual>
-  <collision>
-    <origin xyz="0.12 0.0 -0.395" rpy="0 0 0"/>
-    <geometry>
-      <mesh filename="file://$(find hive_gazebo)/meshes/robots/lidar_link_1.stl" scale="0.001 0.001 0.001"/>
-    </geometry>
-  </collision>
-</link>
-<joint name="robot2_left_wheel_joint" type="continuous">
-  <origin xyz="-1e-06 0.2734 0.0" rpy="0 0 0"/>
-  <parent link="robot2_base_link"/>
-  <child link="robot2_left_wheel"/>
-  <axis xyz="0.0 1.0 0.0"/>
-</joint>
-<joint name="robot2_right_wheel_joint" type="continuous">
-  <origin xyz="-1e-06 -0.2734 0.0" rpy="0 0 0"/>
-  <parent link="robot2_base_link"/>
-  <child link="robot2_right_wheel"/>
-  <axis xyz="0.0 1.0 0.0"/>
-</joint>
-<joint name="robot2_right_caster_joint" type="fixed">
-  <origin xyz="-0.31 -0.19 0.043" rpy="0 0 0"/>
-  <parent link="robot2_base_link"/>
-  <child link="robot2_right_caster"/>
-  <axis xyz="0.0 0.0 -1.0"/>
-</joint>
-<joint name="robot2_left_caster_joint" type="fixed">
-  <origin xyz="-0.31 0.19 0.043" rpy="0 0 0"/>
-  <parent link="robot2_base_link"/>
-  <child link="robot2_left_caster"/>
-  <axis xyz="0.0 0.0 -1.0"/>
-</joint>
-<joint name="robot2_lidar_joint" type="fixed">
-  <origin xyz="-0.12 0.0 0.405" rpy="0 0 0"/>
-  <parent link="robot2_base_link"/>
-  <child link="robot2_lidar_link"/>
-  <axis xyz="-0.0 -0.0 1.0"/>
-</joint>
+<robot name="robot2"
+  xmlns:xacro="http://www.ros.org/wiki/xacro">
+  <xacro:include filename="$(find hive_gazebo)/urdf/robot2/robot2_materials.xacro"/>
+  <xacro:include filename="$(find hive_gazebo)/urdf/robot2/robot2.trans"/>
+  <xacro:include filename="$(find hive_gazebo)/urdf/robot2/robot2.gazebo"/>
+  <link name="robot2_base_link">
+    <inertial>
+      <origin xyz="-0.10420283159261519 -6.650792304374791e-05 0.2749529701185766" rpy="0 0 0"/>
+      <mass value="40.0"/>
+      <inertia ixx="6.809657" iyy="6.121132" izz="6.33059" ixy="0.000377" iyz="-0.000479" ixz="0.18348"/>
+    </inertial>
+    <visual>
+      <origin xyz="0 0 0" rpy="0 0 0"/>
+      <geometry>
+        <mesh filename="file://$(find hive_gazebo)/meshes/robots/base_link.stl" scale="0.001 0.001 0.001"/>
+      </geometry>
+      <material name="blue"/>
+    </visual>
+    <collision>
+      <origin xyz="0 0 0" rpy="0 0 0"/>
+      <geometry>
+        <mesh filename="file://$(find hive_gazebo)/meshes/robots/base_link.stl" scale="0.001 0.001 0.001"/>
+      </geometry>
+    </collision>
+  </link>
+  <link name="robot2_left_wheel">
+    <inertial>
+      <origin xyz="2.6594023369474935e-07 -0.006200652298741449 -4.894162568547244e-09" rpy="0 0 0"/>
+      <mass value="1.3260899817774452"/>
+      <inertia ixx="0.001415" iyy="0.002676" izz="0.001415" ixy="-0.0" iyz="0.0" ixz="0.0"/>
+    </inertial>
+    <visual>
+      <origin xyz="1e-06 -0.277578 0.0" rpy="0 0 0"/>
+      <geometry>
+        <mesh filename="file://$(find hive_gazebo)/meshes/robots/left_wheel_1.stl" scale="0.001 0.001 0.001"/>
+      </geometry>
+      <material name="blue"/>
+    </visual>
+    <collision>
+      <origin xyz="1e-06 -0.277578 0.0" rpy="0 0 0"/>
+      <geometry>
+        <mesh filename="file://$(find hive_gazebo)/meshes/robots/left_wheel_1.stl" scale="0.001 0.001 0.001"/>
+      </geometry>
+    </collision>
+  </link>
+  <link name="robot2_right_wheel">
+    <inertial>
+      <origin xyz="2.5883027950490597e-07 0.006201095560612602 -2.8975644106310483e-10" rpy="0 0 0"/>
+      <mass value="1.3260894987915728"/>
+      <inertia ixx="0.001415" iyy="0.002676" izz="0.001415" ixy="-0.0" iyz="0.0" ixz="-0.0"/>
+    </inertial>
+    <visual>
+      <origin xyz="1e-06 0.269222 0.0" rpy="0 0 0"/>
+      <geometry>
+        <mesh filename="file://$(find hive_gazebo)/meshes/robots/right_wheel_1.stl" scale="0.001 0.001 0.001"/>
+      </geometry>
+      <material name="blue"/>
+    </visual>
+    <collision>
+      <origin xyz="1e-06 0.269222 0.0" rpy="0 0 0"/>
+      <geometry>
+        <mesh filename="file://$(find hive_gazebo)/meshes/robots/right_wheel_1.stl" scale="0.001 0.001 0.001"/>
+      </geometry>
+    </collision>
+  </link>
+  <link name="robot2_right_caster">
+    <inertial>
+      <origin xyz="-0.017519612985357313 2.0677910783639675e-07 -0.05240105157186727" rpy="0 0 0"/>
+      <mass value="1.6117875662608887"/>
+      <inertia ixx="0.001424" iyy="0.001841" izz="0.000923" ixy="-0.0" iyz="-0.0" ixz="-0.000298"/>
+    </inertial>
+    <visual>
+      <origin xyz="0.310001 0.185822 -0.043" rpy="0 0 0"/>
+      <geometry>
+        <mesh filename="file://$(find hive_gazebo)/meshes/robots/right_caster_1.stl" scale="0.001 0.001 0.001"/>
+      </geometry>
+      <material name="blue"/>
+    </visual>
+    <collision>
+      <origin xyz="0.310001 0.185822 -0.043" rpy="0 0 0"/>
+      <geometry>
+        <mesh filename="file://$(find hive_gazebo)/meshes/robots/right_caster_1.stl" scale="0.001 0.001 0.001"/>
+      </geometry>
+    </collision>
+  </link>
+  <link name="robot2_left_caster">
+    <inertial>
+      <origin xyz="-0.017519612985357313 2.0677910747557426e-07 -0.05240105157186712" rpy="0 0 0"/>
+      <mass value="1.6117875662608847"/>
+      <inertia ixx="0.001424" iyy="0.001841" izz="0.000923" ixy="-0.0" iyz="-0.0" ixz="-0.000298"/>
+    </inertial>
+    <visual>
+      <origin xyz="0.310001 -0.194178 -0.043" rpy="0 0 0"/>
+      <geometry>
+        <mesh filename="file://$(find hive_gazebo)/meshes/robots/left_caster_1.stl" scale="0.001 0.001 0.001"/>
+      </geometry>
+      <material name="blue"/>
+    </visual>
+    <collision>
+      <origin xyz="0.310001 -0.194178 -0.043" rpy="0 0 0"/>
+      <geometry>
+        <mesh filename="file://$(find hive_gazebo)/meshes/robots/left_caster_1.stl" scale="0.001 0.001 0.001"/>
+      </geometry>
+    </collision>
+  </link>
+  <link name="robot2_lidar_link">
+    <inertial>
+      <origin xyz="-0.0005135302448306955 -0.0001199429580434408 0.02218628196103728" rpy="0 0 0"/>
+      <mass value="1.4419128562477859"/>
+      <inertia ixx="0.000731" iyy="0.000735" izz="0.000958" ixy="3e-06" iyz="2e-06" ixz="8e-06"/>
+    </inertial>
+    <visual>
+      <origin xyz="0.12 0.0 -0.395" rpy="0 0 0"/>
+      <geometry>
+        <mesh filename="file://$(find hive_gazebo)/meshes/robots/lidar_link_1.stl" scale="0.001 0.001 0.001"/>
+      </geometry>
+      <material name="blue"/>
+    </visual>
+    <collision>
+      <origin xyz="0.12 0.0 -0.395" rpy="0 0 0"/>
+      <geometry>
+        <mesh filename="file://$(find hive_gazebo)/meshes/robots/lidar_link_1.stl" scale="0.001 0.001 0.001"/>
+      </geometry>
+    </collision>
+  </link>
+  <link name="robot2_imu_link"/>
+  <joint name="robot2_imu_joint" type="fixed">
+    <origin xyz="-0.12 0 0.5" rpy="0 0 0"/>
+    <parent link="robot2_base_link"/>
+    <child link="robot2_imu_link"/>
+  </joint>
+  <joint name="robot2_left_wheel_joint" type="continuous">
+    <origin xyz="-1e-06 0.2734 0.0" rpy="0 0 0"/>
+    <parent link="robot2_base_link"/>
+    <child link="robot2_left_wheel"/>
+    <axis xyz="0.0 1.0 0.0"/>
+  </joint>
+  <joint name="robot2_right_wheel_joint" type="continuous">
+    <origin xyz="-1e-06 -0.2734 0.0" rpy="0 0 0"/>
+    <parent link="robot2_base_link"/>
+    <child link="robot2_right_wheel"/>
+    <axis xyz="0.0 1.0 0.0"/>
+  </joint>
+  <joint name="robot2_right_caster_joint" type="fixed">
+    <origin xyz="-0.31 -0.19 0.043" rpy="0 0 0"/>
+    <parent link="robot2_base_link"/>
+    <child link="robot2_right_caster"/>
+    <axis xyz="0.0 0.0 -1.0"/>
+  </joint>
+  <joint name="robot2_left_caster_joint" type="fixed">
+    <origin xyz="-0.31 0.19 0.043" rpy="0 0 0"/>
+    <parent link="robot2_base_link"/>
+    <child link="robot2_left_caster"/>
+    <axis xyz="0.0 0.0 -1.0"/>
+  </joint>
+  <joint name="robot2_lidar_joint" type="fixed">
+    <origin xyz="-0.12 0.0 0.405" rpy="0 0 0"/>
+    <parent link="robot2_base_link"/>
+    <child link="robot2_lidar_link"/>
+    <axis xyz="-0.0 -0.0 1.0"/>
+  </joint>
 </robot>
