Commit message: refact: change camera's fov and z value for realistic test.

File: hive_gazebo/urdf/simple_cameras/camera1.urdf (robot description, URDF)
Before this commit: robot camera1, 3 links, 2 joints
Joints:
- joint world_ceiling_joint: origin xyz=0 0 3.505 rpy=0 0 0 -> xyz=0 0 2.5 rpy=0 0 0

File: hive_gazebo/urdf/simple_cameras/camera2.urdf (robot description, URDF)
Before this commit: robot camera2, 3 links, 2 joints
Joints:
- joint world_ceiling_joint: origin xyz=0 0 3.505 rpy=0 0 0 -> xyz=0 0 2.5 rpy=0 0 0

Commit message: feat: add number world.

File: hive_gazebo/urdf/simple_cameras/camera1.urdf (robot description, URDF)
Before this commit: robot camera1, 3 links, 2 joints
Joints:
- joint world_ceiling_joint: origin xyz=0 0 2.5 rpy=0 0 0 -> xyz=0 0 5 rpy=0 0 0

File: hive_gazebo/urdf/simple_cameras/camera2.urdf (robot description, URDF)
Before this commit: robot camera2, 3 links, 2 joints
Joints:
- joint world_ceiling_joint: origin xyz=0 0 2.5 rpy=0 0 0 -> xyz=0 0 5 rpy=0 0 0
